Commit message: URDF changes to include microstrain's IMU

File: jackal_description/urdf/jackal.urdf.xacro (robot description, xacro)
@@ -122,5 +122,5 @@
        always points to the "active" IMU. When an upgrade IMU is connected, the
        internal_imu_link should remain, but imu_link should point to the upgrade one. -->
-  <link name="imu_link">
+  <link name="internal_imu_link">
     <inertial>
       <mass value="0.001"/>
@@ -129,7 +129,7 @@
     </inertial>
   </link>
-  <joint name="imu_joint" type="fixed">
+  <joint name="internal_imu_joint" type="fixed">
     <parent link="chassis_link" />
-    <child link="imu_link" />
+    <child link="internal_imu_link" />
   </joint>
   <!-- TODO: Same note as applies to imu_link -->
@@ -174,3 +174,4 @@
   <!-- Optional custom includes. -->
   <xacro:include filename="$(optenv JACKAL_URDF_EXTRAS empty.urdf)" />
+  <xacro:include filename="$(optenv JACKAL_URDF_EXTRAS microstrain_imu.urdf)" />
 </robot>
